Commit message: changed ur_robots macro origin

File: my_robot_cell/my_robot_cell_description/urdf/my_robot_cell.urdf.xacro (robot description, xacro)
@@ -72,5 +72,5 @@
     <parent link="table"/>
     <child link="robot_mount"/>
-    <origin xyz="0.845 0.9 0" rpy="0 0 0" />
+    <origin xyz="0.845 0.85 0" rpy="0 0 ${pi}" />
   </joint>
   <xacro:ur_robot
@@ -87,5 +87,5 @@
     input_recipe_filename="$(arg ur_input_recipe_filename)"
   >
-    <origin xyz="0 -0.05 0" rpy="0 0 ${pi}" />
+    <origin xyz="0 0 0" rpy="0 0 0" />
   </xacro:ur_robot>
 </robot>

Commit message: Revert "adapted tutorial to new ur_description"
This reverts commit 2fa0628090c62d7be474aaf7eaa0edb934422c86.

File: my_robot_cell/my_robot_cell_description/urdf/my_robot_cell.urdf.xacro (robot description, xacro)
@@ -2,19 +2,88 @@
 <robot name="my_robot_cell" xmlns:xacro="http://ros.org/wiki/xacro">
   <xacro:include filename="$(find ur_description)/urdf/ur_macro.xacro"/>
-  <xacro:include filename="$(find my_robot_cell_description)/urdf/my_robot_cell_macro.xacro"/>
   <xacro:arg name="ur_type" default="ur20"/>
+  <xacro:arg name="robot_ip" default="0.0.0.0"/>
   <xacro:arg name="joint_limit_params" default="$(find ur_description)/config/$(arg ur_type)/joint_limits.yaml"/>
   <xacro:arg name="kinematics_params" default="$(find ur_description)/config/$(arg ur_type)/default_kinematics.yaml"/>
   <xacro:arg name="physical_params" default="$(find ur_description)/config/$(arg ur_type)/physical_parameters.yaml"/>
   <xacro:arg name="visual_params" default="$(find ur_description)/config/$(arg ur_type)/visual_parameters.yaml"/>
-  <xacro:my_robot_cell/>
+  <xacro:arg name="ur_script_filename" default="$(find ur_client_library)/resources/external_control.urscript"/>
+  <xacro:arg name="ur_output_recipe_filename" default="$(find ur_robot_driver)/resources/rtde_input_recipe.txt"/>
+  <xacro:arg name="ur_input_recipe_filename" default="$(find ur_robot_driver)/resources/rtde_output_recipe.txt"/>
+  <link name="world"/>
+  <joint name="table_to_world" type="fixed">
+    <parent link="world"/>
+    <child link="table"/>
+    <origin xyz="0 0 1"/>
+  </joint>
+  <link name="table">
+    <visual>
+      <geometry>
+        <mesh filename="package://my_robot_cell_description/meshes/fzi_table.dae"/>
+      </geometry>
+      <origin rpy="0 0 0" xyz="0.75 0.5 -1"/>
+    </visual>
+    <collision>
+      <geometry>
+        <mesh filename="package://my_robot_cell_description/meshes/fzi_table.dae"/>
+      </geometry>
+      <origin rpy="0 0 0" xyz="0.75 0.5 -1"/>
+    </collision>
+  </link>
+  <link name="monitor">
+    <visual>
+      <geometry>
+        <mesh filename="package://my_robot_cell_description/meshes/171005_Motek_Monitor_L.dae"/>
+      </geometry>
+    </visual>
+    <collision>
+      <geometry>
+        <mesh filename="package://my_robot_cell_description/meshes/171005_Motek_Monitor_L.dae"/>
+      </geometry>
+    </collision>
+  </link>
+  <joint name="base_to_monitor" type="fixed">
+    <parent link="table"/>
+    <child link="monitor"/>
+    <origin xyz="0.2 0.6 0"/>
+  </joint>
+  <material name="white">
+    <color rgba="1 1 1 1"/>
+  </material>
+  <link name="wall">
+    <visual>
+      <geometry>
+        <mesh filename="package://my_robot_cell_description/meshes/wall.dae"/>
+      </geometry>
+    </visual>
+    <collision>
+      <geometry>
+        <box size="4.44 0.1 2.5"/>
+      </geometry>
+    </collision>
+  </link>
+  <joint name="base_to_wall" type="fixed">
+    <parent link="table"/>
+    <child link="wall"/>
+    <origin xyz="1.25 1.5 0.5"/>
+  </joint>
+  <link name="robot_mount"/>
+  <joint name="base_to_robot_mount" type="fixed">
+    <parent link="table"/>
+    <child link="robot_mount"/>
+    <origin xyz="0.845 0.85 0" rpy="0 0 ${pi}" />
+  </joint>
   <xacro:ur_robot
     name="$(arg ur_type)"
     tf_prefix="$(arg ur_type)_"
     parent="robot_mount"
+    robot_ip="$(arg robot_ip)"
     joint_limits_parameters_file="$(arg joint_limit_params)"
     kinematics_parameters_file="$(arg kinematics_params)"
     physical_parameters_file="$(arg physical_params)"
     visual_parameters_file="$(arg visual_params)"
+    script_filename="$(arg ur_script_filename)"
+    output_recipe_filename="$(arg ur_output_recipe_filename)"
+    input_recipe_filename="$(arg ur_input_recipe_filename)"
   >
     <origin xyz="0 0 0" rpy="0 0 0" />

Commit message: Update custom workspace example to latest changes

File: my_robot_cell/my_robot_cell_description/urdf/my_robot_cell.urdf.xacro (robot description, xacro)
@@ -1,22 +1,21 @@
 <?xml version="1.0"?>
 <robot name="my_robot_cell" xmlns:xacro="http://ros.org/wiki/xacro">
-  <xacro:include filename="$(find ur_description)/urdf/ur_macro.xacro"/>
   <xacro:include filename="$(find my_robot_cell_description)/urdf/my_robot_cell_macro.xacro"/>
   <xacro:arg name="ur_type" default="ur20"/>
-  <xacro:arg name="joint_limit_params" default="$(find ur_description)/config/$(arg ur_type)/joint_limits.yaml"/>
-  <xacro:arg name="kinematics_params" default="$(find ur_description)/config/$(arg ur_type)/default_kinematics.yaml"/>
-  <xacro:arg name="physical_params" default="$(find ur_description)/config/$(arg ur_type)/physical_parameters.yaml"/>
-  <xacro:arg name="visual_params" default="$(find ur_description)/config/$(arg ur_type)/visual_parameters.yaml"/>
-  <xacro:my_robot_cell/>
-  <xacro:ur_robot
-    name="$(arg ur_type)"
-    tf_prefix="$(arg ur_type)_"
-    parent="robot_mount"
-    joint_limits_parameters_file="$(arg joint_limit_params)"
-    kinematics_parameters_file="$(arg kinematics_params)"
-    physical_parameters_file="$(arg physical_params)"
-    visual_parameters_file="$(arg visual_params)"
-  >
-    <origin xyz="0 0 0" rpy="0 0 0" />
-  </xacro:ur_robot>
+  <xacro:arg name="joint_limits_parameters_file" default="$(find ur_description)/config/$(arg ur_type)/joint_limits.yaml"/>
+  <xacro:arg name="kinematics_parameters_file" default="$(find ur_description)/config/$(arg ur_type)/default_kinematics.yaml"/>
+  <xacro:arg name="physical_parameters_file" default="$(find ur_description)/config/$(arg ur_type)/physical_parameters.yaml"/>
+  <xacro:arg name="visual_parameters_file" default="$(find ur_description)/config/$(arg ur_type)/visual_parameters.yaml"/>
+  <link name="world"/>
+  <!--This will create the scene where the robot is located in-->
+  <xacro:my_robot_cell
+    parent="world"
+    ur_type="$(arg ur_type)"
+    joint_limits_parameters_file="$(arg joint_limits_parameters_file)"
+    kinematics_parameters_file="$(arg kinematics_parameters_file)"
+    physical_parameters_file="$(arg physical_parameters_file)"
+    visual_parameters_file="$(arg visual_parameters_file)"
+    >
+      <origin xyz="0 0 1" rpy="0 0 0" />
+  </xacro:my_robot_cell>
 </robot>

File: my_robot_cell/my_robot_cell_description/urdf/my_robot_cell_macro.xacro (robot description, xacro)
@@ -1,10 +1,18 @@
 <?xml version="1.0"?>
 <robot xmlns:xacro="http://ros.org/wiki/xacro">
-  <xacro:macro name="my_robot_cell">
-    <link name="world"/>
-    <joint name="table_to_world" type="fixed">
-      <parent link="world"/>
-      <child link="table"/>
-      <origin xyz="0 0 1"/>
+  <xacro:include filename="$(find ur_description)/urdf/ur_macro.xacro"/>
+  <xacro:macro name="my_robot_cell" params="
+    parent
+    *origin
+    ur_type
+    joint_limits_parameters_file
+    kinematics_parameters_file
+    physical_parameters_file
+    visual_parameters_file
+    ">
+    <joint name="table_base_joint" type="fixed">
+      <xacro:insert_block name="origin" />
+      <parent link="${parent}" />
+      <child link="table" />
     </joint>
     <link name="table">
@@ -65,4 +73,16 @@
       <origin xyz="0.845 0.85 0" rpy="0 0 ${pi}" />
     </joint>
+    <!--This will create the specific robot-->
+    <xacro:ur_robot
+      name="${ur_type}"
+      tf_prefix="${ur_type}_"
+      parent="robot_mount"
+      joint_limits_parameters_file="${joint_limits_parameters_file}"
+      kinematics_parameters_file="${kinematics_parameters_file}"
+      physical_parameters_file="${physical_parameters_file}"
+      visual_parameters_file="${visual_parameters_file}"
+    >
+      <origin xyz="0 0 0" rpy="0 0 0" />
+    </xacro:ur_robot>
   </xacro:macro>
 </robot>
